Commit message: 2022.08.06

File: assets/urdf/hyper.urdf (robot description, URDF)
Before this commit: robot hyper, 14 links, 13 joints
Joints:
- joint LB_joint1: origin xyz=-0.1025 0.04025 -0.00175 rpy=-1.57 0 0 -> xyz=-0.1025 0.04025 -0.00175 rpy=0 0 0
- joint LF_joint1: origin xyz=0.1515 0.04025 -0.00175 rpy=-1.57 0 0 -> xyz=0.1515 0.04025 -0.00175 rpy=0 0 0
- joint RB_joint1: origin xyz=-0.1025 -0.04025 -0.00175 rpy=-1.57 0 0 -> xyz=-0.1025 -0.04025 -0.00175 rpy=0 0 0
- joint RF_joint1: origin xyz=0.1515 -0.00175 0.04025 rpy=0 0 0 -> xyz=0.1515 -0.04025 -0.00175 rpy=0 0 0
- joint planar: origin xyz=0.0 0.0 0.0 rpy=-1.57 0 0 -> xyz=0.0 0.0 0.0 rpy=0 0 0

File: assets/urdf/manipulator1.urdf (robot description, URDF)
Before this commit: robot manipulator1, 2 links, 1 joints
Links:
- removed link base_link
- removed link link1_link
- added link base, mass 0.098358; collision mesh filename=../meshes/base_link.STL; visual mesh filename=../meshes/base_link.STL
- added link link1, mass 0.12845; collision mesh filename=../meshes/link1_link.STL; visual mesh filename=../meshes/link1_link.STL
Joints:
- joint joint1: child link1_link -> link1; parent base_link -> base
